Commit message: <feat> real deploy test with gimbal identified system

File: robots/beetle_omni/beetle_omni.urdf (robot description, URDF)
Before this commit: robot beetle-art-omni, 22 links, 21 joints
Joints:
- joint gimbal1: limit lower=-3.926991 upper=3.926991 effort=6.6 velocity=3.0 -> lower=-7.926991 upper=7.926991 effort=3.0 velocity=10.0
- joint gimbal2: limit lower=-3.926991 upper=3.926991 effort=6.6 velocity=3.0 -> lower=-7.926991 upper=7.926991 effort=3.0 velocity=10.0
- joint gimbal3: limit lower=-3.926991 upper=3.926991 effort=6.6 velocity=3.0 -> lower=-7.926991 upper=7.926991 effort=3.0 velocity=10.0
- joint gimbal4: limit lower=-3.926991 upper=3.926991 effort=6.6 velocity=3.0 -> lower=-7.926991 upper=7.926991 effort=3.0 velocity=10.0
