Commit message: <perf> perf for realworld deploy

File: robots/beetle_omni/urdf/beetle_art_omni.urdf.xacro (robot description, xacro)
@@ -130,5 +130,5 @@
       <origin rpy="0 0 0" xyz="0 0 0"/>
       <axis xyz="1 0 0"/>
-      <dynamics damping="0.8" friction="0.0"/>
+      <dynamics damping="0.0" friction="0.0"/>
     </joint>
     <transmission name="joint_tran${self}">

Commit message: <fix> fix bug on joint parameters and add doc
1. modify joint parameters for real2sim
2. add doc for foxglove installation

File: robots/beetle_omni/urdf/beetle_art_omni.urdf.xacro (robot description, xacro)
@@ -116,7 +116,7 @@
         <mass value="0.005"/>
         <inertia
-            ixx="0.001" ixy="0.0" ixz="0.0"
-            iyy="0.001" iyz="0.0"
-            izz="0.001"/>
+            ixx="0.00001" ixy="0.0" ixz="0.0"
+            iyy="0.00001" iyz="0.0"
+            izz="0.00001"/>
       </inertial>
     </link>
@@ -125,5 +125,5 @@
     #### gimbal joints ####
     <joint name="gimbal${self}" type="revolute">
-      <limit effort="6.6" lower="-3.926991" upper="3.926991" velocity="3.0"/>
+      <limit effort="3.0" lower="-7.926991" upper="7.926991" velocity="10.0"/>
       <parent link="rotor_arm${self}"/>
       <child link="gimbal_link${self}"/>

Commit message: <feat> experiments arrange code
1. add safety structure
2. add pub_waypoints.py to pub desired pose sequence
3. add pub_trajectory.py to pub desired pose trajectory

File: robots/beetle_omni/urdf/beetle_art_omni.urdf.xacro (robot description, xacro)
@@ -31,4 +31,57 @@
       <origin rpy="0 0 0" xyz="0 0 0"/>
     </joint>
+    <!-- <link
+    name="safety_link">
+    <inertial>
+      <origin
+        xyz="1.9934E-06 2.1863E-06 0.025823"
+        rpy="0 0 0" />
+      <mass
+        value="0.5315" />
+      <inertia
+        ixx="0.0057039"
+        ixy="1.2576E-10"
+        ixz="8.5498E-13"
+        iyy="0.005704"
+        iyz="-5.6396E-11"
+        izz="0.0106" />
+    </inertial>
+    <visual>
+      <origin
+        xyz="0 0 0"
+        rpy="0 0 0" />
+      <geometry>
+        <mesh
+          filename="package://beetle_omni/urdf/mesh/safety_link.STL" />
+      </geometry>
+      <material
+        name="">
+        <color
+          rgba="0.26863 1 0.26863 1" />
+      </material>
+    </visual>
+    <collision>
+      <origin
+        xyz="0 0 0"
+        rpy="0 0 0" />
+      <geometry>
+        <mesh
+          filename="package://beetle_omni/urdf/mesh/safety_link.STL" />
+      </geometry>
+    </collision>
+  </link>
+  <joint
+    name="safety"
+    type="fixed">
+    <origin
+      xyz="0 0 0"
+      rpy="0 0 0" />
+    <parent
+      link="root" />
+    <child
+      link="safety_link" />
+    <axis
+      xyz="0 0 0" />
+  </joint> -->
     ## fc: flight controller. Note that "baselink" is assigned to "fc" in common.xacro by default
     <link name="fc">

Commit message: <policy> add policy and add trajectory loop

File: robots/beetle_omni/urdf/beetle_art_omni.urdf.xacro (robot description, xacro)
@@ -178,5 +178,5 @@
     #### gimbal joints ####
     <joint name="gimbal${self}" type="revolute">
-      <limit effort="3.0" lower="-7.926991" upper="7.926991" velocity="10.0"/>
+      <limit effort="3.0" lower="-3.5" upper="3.5" velocity="10.0"/>
       <parent link="rotor_arm${self}"/>
       <child link="gimbal_link${self}"/>

Commit message: <policy>

File: robots/beetle_omni/urdf/beetle_art_omni.urdf.xacro (robot description, xacro)
@@ -178,5 +178,5 @@
     #### gimbal joints ####
     <joint name="gimbal${self}" type="revolute">
-      <limit effort="3.0" lower="-3.5" upper="3.5" velocity="10.0"/>
+      <limit effort="3.0" lower="-6.9" upper="6.9" velocity="10.0"/>
       <parent link="rotor_arm${self}"/>
       <child link="gimbal_link${self}"/>
