Commit message: <test> rebuttal for 90 pitch, baseline training
just want to deploy in real-world and try to make 90 or 180 pitch

File: robots/beetle_omni/urdf/beetle_rl.urdf.xacro (robot description, xacro)
@@ -79,5 +79,5 @@
       xyz="0 0 0" />
   </joint>
-  <!-- <link
+  <link
     name="battery_link">
     <inertial>
@@ -126,5 +126,5 @@
     <axis
       xyz="0 0 0" />
-  </joint> -->
+  </joint>
     ## fc: flight controller. Note that "baselink" is assigned to "fc" in common.xacro by default
     <link name="fc">

Commit message: <policy> add fault tolerant policy

File: robots/beetle_omni/urdf/beetle_rl.urdf.xacro (robot description, xacro)
@@ -79,5 +79,5 @@
       xyz="0 0 0" />
   </joint>
-  <link
+  <!-- <link
     name="battery_link">
     <inertial>
@@ -126,5 +126,5 @@
     <axis
       xyz="0 0 0" />
-  </joint>
+  </joint> -->
     ## fc: flight controller. Note that "baselink" is assigned to "fc" in common.xacro by default
     <link name="fc">
